File: soc-module/soc-module/soc-module.kicad_pcb (KiCad board)
At the start: 2 copper layers, 11 parts, among them J1 Micro_SD_Card, J2 Conn_01x13, J3 Conn_01x14, U1 ATECC608A-SSHDA, U2 ESP32-WROVER-IE-16MB

Commit message: SoC Module Work On
Parts:
- added R3: R, Resistor_SMD:R_1206_3216Metric_Pad1.30x1.75mm_HandSolder, B.Cu at (126.5, 88.0)
- added R4: R, Resistor_SMD:R_1206_3216Metric_Pad1.30x1.75mm_HandSolder, B.Cu at (126.5, 91.7)
- added R5: R, Resistor_SMD:R_1206_3216Metric_Pad1.30x1.75mm_HandSolder, B.Cu at (126.5, 95.4)
- added R6: R, Resistor_SMD:R_1206_3216Metric_Pad1.30x1.75mm_HandSolder, B.Cu at (126.5, 99.1)
- added SW1: Prog, footprints:SW4SMD_63X161LS, F.Cu at (126.0, 108.0)
- added SW2: Reset, footprints:SW4SMD_63X161LS, F.Cu at (126.0, 103.0)
- J1: value Micro_SD_Card -> Micro_SD_Card_Det_Hirose_DM3AT; footprint footprints:HRS_DM3AT-SF-PEJM5 -> Connector_Card:microSD_HC_Hirose_DM3AT-SF-PEJM5
- moved C2 15.8 mm to (141.3, 104.5)
- moved C1 13.9 mm to (141.3, 100.8), turned to 180 degrees
- moved J1 7.81 mm to (129.5, 92.4)
- moved R2 5.10 mm to (141.3, 93.5), turned to 180 degrees
- moved R1 2.20 mm to (141.3, 97.2)
- moved C4 1.82 mm to (141.3, 89.9), turned to 180 degrees
- moved C3 0.80 mm to (141.3, 86.2), turned to 180 degrees
- moved J2 0.30 mm to (164.5, 108.5)
- moved J3 0.30 mm to (164.5, 82.5)
- moved U1 0.22 mm to (134.6, 103.3), turned to 0 degrees
Connections:
- J1 pad 2: Net-(J1-Pad2) -> IO5
- J1 pad 3: Net-(J1-Pad3) -> SPI_0_MOSI
- J1 pad 5: Net-(J1-Pad5) -> SPI_0_CLK
- J1 pad 7: Net-(J1-Pad7) -> SPI_0_MISO
- J2 pad 3: IO22 -> I2C_SCL
- J2 pad 6: IO21 -> I2C_SDA
- U1 pad 5: Net-(U1-Pad5) -> I2C_SDA
- U1 pad 6: Net-(U1-Pad6) -> I2C_SCL
- U2 pad 33: IO21 -> I2C_SDA
- U2 pad 36: IO22 -> I2C_SCL
Routing:
- net +3V3: track 0.00 -> 88.2 mm, vias 0 -> 2
- net Chip_PU: track 0.00 -> 80.5 mm, vias 0 -> 2
- net I2C_SCL: track 0.00 -> 54.1 mm, vias 0 -> 2
- net I2C_SDA: track 0.00 -> 53.1 mm, vias 0 -> 2
- net IO0: track 0.00 -> 45.4 mm, vias 0 -> 1
- net IO5: track 0.00 -> 32.3 mm, vias 0 -> 2
- net IO18: track 0.00 -> 20.0 mm, vias 0 -> 1
- net IO4: track 0.00 -> 19.8 mm, vias 0 -> 1
- net IO19: track 0.00 -> 19.1 mm, vias 0 -> 1
- net U0RXD: track 0.00 -> 18.6 mm, vias 0 -> 1
- net U0TXD: track 0.00 -> 17.5 mm, vias 0 -> 1
- net IO23: track 0.00 -> 15.3 mm, vias 0 -> 1
- net SPI_0_MOSI: track 0.00 -> 10.2 mm, vias 0 -> 1
- net SPI_0_CLK: track 0.00 -> 9.56 mm, vias 0 -> 1
- net SPI_0_MISO: track 0.00 -> 9.38 mm, vias 0 -> 1
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Other:
- board outline added: 56 x 31 mm
- board text added: "Satellite SoC Module v2.0 GrayC GmbH"
- board text added: "TOP"

Commit message: Ongoing Work Metering Module
Parts:
- renumbered C1 to C1^
Routing:
- net IO5: track 32.3 -> 61.1 mm, vias 2 -> 3
- net IO13: track 3.50 -> 26.7 mm
- net IO12: track 3.53 -> 25.2 mm
- net IO14: track 3.52 -> 23.9 mm
- net IO27: track 3.51 -> 23.0 mm
- net IO26: track 3.50 -> 21.9 mm
- net IO25: track 3.52 -> 21.0 mm
- net IO33: track 3.51 -> 19.8 mm
- net IO32: track 3.50 -> 19.0 mm
- net I35: track 3.53 -> 17.9 mm
- net I34: track 3.52 -> 16.9 mm
- net I39: track 3.50 -> 15.7 mm
- net I36: track 3.51 -> 14.6 mm
- net Chip_PU: track 80.5 -> 90.8 mm
- net +3V3: track 88.2 -> 97.3 mm
Other:
- board text added: "BOT"
- board text added: "WiFi"
