File: soc-module/soc-module.kicad_pcb (KiCad board)
At the start: 2 copper layers, 56 x 31 mm, 17 parts, among them J1 Micro_SD_Card_Det_Hirose_DM3AT, J2 Conn_01x13, J3 Conn_01x14, SW1 Prog, SW2 Reset, U1 ATECC608A-SSHDA, U2 ESP32-WROVER-IE-16MB

Commit message: Ongoing
Parts:
- C1: renamed from C1^; value C -> 100nF
- C2, C3, C4: value C -> 100nF
- J1: value Micro_SD_Card_Det_Hirose_DM3AT -> Micro_SD
- J2: value Conn_01x13 -> East
- J3: value Conn_01x14 -> West
- R1, R2, R3, R4, R5, R6: value R -> 10k
- turned R1 to 180 degrees
Connections:
- R1 pad 1: +3V3 -> IO0
- R1 pad 2: IO0 -> +3V3
