File: development-board/development-board.sch (KiCad schematic (older format))
At the start: 5 parts

Commit message: Ongoing Work. Still not ready for small and dedicated commits.
Parts:
- removed J?: Conn_02x10_Odd_Even, symbol Connector_Generic:Conn_02x10_Odd_Even
- removed J?: USB_B, symbol Connector:USB_B
- removed J?: RJ12, symbol Connector:RJ12
- removed U?: FT232H, symbol Interface_USB:FT232H
- removed U?: M93C46-WMN6TP, SOIC127P600X175-8N, symbol M93C46-WMN6TP:M93C46-WMN6TP
- added C4: 100nF, Capacitor_SMD:C_1206_3216Metric_Pad1.33x1.80mm_HandSolder, symbol Device:C
- added C5: 10uF, Capacitor_SMD:C_1206_3216Metric_Pad1.33x1.80mm_HandSolder, symbol Device:C
- added C6, C7: C, Capacitor_SMD:C_1206_3216Metric_Pad1.33x1.80mm_HandSolder, symbol Device:C
- added D1: BZT52C6V2, Diode_SMD:D_SOD-323_HandSoldering, symbol Device:D_TVS
- added D2: 1N5819, Diode_SMD:D_SOD-323_HandSoldering, symbol Diode:1N5819
- added D3: Power, LED_SMD:LED_1206_3216Metric_Pad1.42x1.75mm_HandSolder, symbol Device:LED
- added D6: TXD, LED_SMD:LED_1206_3216Metric_Pad1.42x1.75mm_HandSolder, symbol Device:LED
- added D7: RXD, LED_SMD:LED_1206_3216Metric_Pad1.42x1.75mm_HandSolder, symbol Device:LED
- added D8: Status, LED_SMD:LED_1206_3216Metric_Pad1.42x1.75mm_HandSolder, symbol Device:LED
- added F1: 6V/800mA, Fuse:Fuse_1206_3216Metric_Pad1.42x1.75mm_HandSolder, symbol Device:Fuse
- added H1, H2, H3, H4: MountingHole_Pad, MountingHole:MountingHole_3.2mm_M3_DIN965_Pad, symbol Mechanical:MountingHole_Pad
- added H5: WiFi Cable, MountingHole:MountingHole_5.5mm, symbol Mechanical:MountingHole
- added H6: Antenna, MountingHole:MountingHole_5.5mm, symbol Mechanical:MountingHole
- added J1: East, Connector_PinHeader_2.54mm:PinHeader_1x14_P2.54mm_Vertical, symbol Connector_Generic:Conn_01x14
- added J10: Ext_5V, Connector_PinHeader_2.54mm:PinHeader_1x02_P2.54mm_Horizontal, symbol Connector_Generic:Conn_01x02
- added J8: West, Connector_PinHeader_2.54mm:PinHeader_1x14_P2.54mm_Vertical, symbol Connector_Generic:Conn_01x14
- added J9: PinOut, Connector_PinHeader_2.54mm:PinHeader_2x14_P2.54mm_Vertical, symbol Connector_Generic:Conn_02x14_Odd_Even
- added Q3, Q4: S8050, Package_TO_SOT_SMD:SOT-23, symbol Transistor_BJT:S8050
- added R25, R34, R35, R36, R37: 10k, Resistor_SMD:R_1206_3216Metric_Pad1.30x1.75mm_HandSolder, symbol Device:R
- added R26, R31, R32, R33: 220R, Resistor_SMD:R_1206_3216Metric_Pad1.30x1.75mm_HandSolder, symbol Device:R
- added SW1: Reset, Button_Switch_SMD:SW_SPST_PTS645, symbol Switch:SW_Push
- added SW2: Setup, Button_Switch_SMD:SW_SPST_PTS645, symbol Switch:SW_Push
- added SW3: Power, Button_Switch_THT:SW_E-Switch_EG1224_SPDT_Angled, symbol Switch:SW_SPDT
- added U1: LD1117S33, Package_TO_SOT_SMD:SOT-223-3_TabPin2, symbol Regulator_Linear:LD1117S33TR_SOT223
Connections:
- new net: D3.2 (A), R26.2
- new net: Q4.2 (B), R37.2
- new net: Q3.2 (B), R36.1
- new net: D1.1 (A1), D2.2 (A), F1.2, R25.1
- new net: F1.1, SW3.2 (B)
- new net: J10.1 (Pin_1), SW3.1 (A)
- new net: D6.2 (A), R31.2
- new net: D7.2 (A), R32.2
- new net: D8.2 (A), R33.2
- new net +3V3: C5.1, J8.1 (Pin_1), J9.1 (Pin_1), R26.1, R31.1, R32.1, R34.1, R35.1, U1.2 (VO)
- new net +5V: C4.1, D2.1 (K), J9.2 (Pin_2), U1.3 (VI)
- new net Chip_PU: C6.1, J8.2 (Pin_2), J9.3 (Pin_3), Q4.3 (C), R34.2, SW1.2
- new net FT_~DTR~: Q3.1 (E), R37.1
- new net FT_~RTS~: Q4.1 (E), R36.2
- new net GND: C4.2, C5.2, C6.2, C7.2, D1.2 (A2), D3.1 (K), D8.1 (K), H1.1, H2.1, H3.1, H4.1, J1.1 (Pin_1), J1.14 (Pin_14), J10.2 (Pin_2), J9.28 (Pin_28), R25.2, SW1.1, SW2.1, U1.1 (GND)
- new net I34: J8.5 (Pin_5), J9.9 (Pin_9)
- new net I35: J8.6 (Pin_6), J9.11 (Pin_11)
- new net I36: J8.3 (Pin_3), J9.5 (Pin_5)
- new net I39: J8.4 (Pin_4), J9.7 (Pin_7)
- new net IO0: C7.1, J1.11 (Pin_11), J9.22 (Pin_22), Q3.3 (C), R35.2, SW2.2
- new net IO12: J8.13 (Pin_13), J9.25 (Pin_25)
- new net IO13: J8.14 (Pin_14), J9.27 (Pin_27), R33.1
- new net IO14: J8.12 (Pin_12), J9.23 (Pin_23)
- new net IO15: J1.13 (Pin_13), J9.26 (Pin_26)
- new net IO18: J1.8 (Pin_8), J9.16 (Pin_16)
- new net IO19: J1.7 (Pin_7), J9.14 (Pin_14)
- new net IO2: J1.12 (Pin_12), J9.24 (Pin_24)
- new net IO21: J1.6 (Pin_6), J9.12 (Pin_12)
- new net IO22: J1.3 (Pin_3), J9.6 (Pin_6)
- new net IO23: J1.2 (Pin_2), J9.4 (Pin_4)
- new net IO25: J8.9 (Pin_9), J9.17 (Pin_17)
- new net IO26: J8.10 (Pin_10), J9.19 (Pin_19)
- new net IO27: J8.11 (Pin_11), J9.21 (Pin_21)
- new net IO32: J8.7 (Pin_7), J9.13 (Pin_13)
- new net IO33: J8.8 (Pin_8), J9.15 (Pin_15)
- new net IO4: J1.10 (Pin_10), J9.20 (Pin_20)
- new net IO5: J1.9 (Pin_9), J9.18 (Pin_18)
- new net RX_LED: D7.1 (K)
- new net TX_LED: D6.1 (K)
- new net U0RXD: J1.5 (Pin_5), J9.10 (Pin_10)
- new net U0TXD: J1.4 (Pin_4), J9.8 (Pin_8)
- new net VBUS: SW3.3 (C)
