File: nbiot-extension/nbiot-extension.sch (KiCad schematic (older format))
At the start: 2 parts

Commit message: NB IoT ongoing work
Parts:
- removed U?: SARA-U201, RF_GSM:ublox_SARA-G3_LGA-96, symbol RF_GSM:SARA-U201
- added U1: BC66NB-04-STD, XCVR_BC66NB-04-STD, symbol BC66NB-04-STD:BC66NB-04-STD
- gave numbers to parts that had none: 1
Connections:
- new net: U1.1 (GND), U1.27 (GND), U1.34 (GND), U1.36 (GND), U1.37 (GND), U1.40 (GND), U1.41 (GND)
- new net: U1.2 (RESERVED), U1.21 (RESERVED), U1.22 (RESERVED), U1.23 (RESERVED), U1.25 (RESERVED), U1.26 (RESERVED), U1.3 (RESERVED), U1.30 (RESERVED), U1.31 (RESERVED), U1.32 (RESERVED), U1.33 (RESERVED), U1.4 (RESERVED), U1.44 (RESERVED), U1.45 (RESERVED), U1.46 (RESERVED), U1.48 (RESERVED), U1.5 (RESERVED), U1.52 (RESERVED), U1.53 (RESERVED), U1.54 (RESERVED), U1.55 (RESERVED), U1.56 (RESERVED), U1.57 (RESERVED), U1.58 (RESERVED), U1.6 (RESERVED), U1.8 (RESERVED)
Changed lines of the file:
@@
 $EndDescr
 $Comp
-L RF_GSM:SARA-U201 U?
-U 1 1 61C20FD4
-P 4750 3250
-F 0 "U?" H 4750 2061 50  0000 C CNN
-F 1 "SARA-U201" H 4750 1970 50  0000 C CNN
-F 2 "RF_GSM:ublox_SARA-G3_LGA-96" H 5450 2200 50  0001 C CNN
-F 3 "https://www.u-blox.com/sites/default/files/SARA-U2_DataSheet_(UBX-13005287).pdf" H 4750 3250 50  0001 C CNN
-	1    4750 3250
-	1    0    0    -1
-$EndComp
-$Comp
-L Connector:SIM_Card_Shielded J?
+L Connector:SIM_Card_Shielded J1
 U 1 1 61C22CA2
 P 7100 2650
-F 0 "J?" H 7730 2700 50  0000 L CNN
+F 0 "J1" H 7730 2700 50  0000 L CNN
 F 1 "SIM_Card_Shielded" H 7730 2609 50  0000 L CNN
 F 2 "Connector_Card:microSIM_JAE_SF53S006VCBR2000" H 7100 3000 50  0001 C CNN
@@
 	1    0    0    -1
 $EndComp
+$Comp
+L BC66NB-04-STD:BC66NB-04-STD U1
+U 1 1 62309D67
+P 4100 3650
+F 0 "U1" H 4100 5017 50  0000 C CNN
+F 1 "BC66NB-04-STD" H 4100 4926 50  0000 C CNN
+F 2 "XCVR_BC66NB-04-STD" H 4100 3650 50  0001 L BNN
+F 3 "" H 4100 3650 50  0001 L BNN
+F 4 "BC66" H 4100 3650 50  0001 L BNN "MP"
+F 5 "Unavailable" H 4100 3650 50  0001 L BNN "AVAILABILITY"
+F 6 "BC66 is a high-performance, multi-band LTE Cat NB-IoT module with extremely low power consumption. The ultra-compact 17.7mm × 15.8mm × 2.0mm profile makes it the perfect choice for size sensitive applications" H 4100 3650 50  0001 L BNN "DESCRIPTION"
+F 7 "None" H 4100 3650 50  0001 L BNN "PRICE"
+F 8 "Radial Vertical Cylinder  Quectel Wireless Solutions Co., Ltd" H 4100 3650 50  0001 L BNN "PACKAGE"
+F 9 "Quectel Wireless Solutions Co., Ltd" H 4100 3650 50  0001 L BNN "MF"
+	1    4100 3650
+	1    0    0    -1
+$EndComp
