File: panel-module/panel-module.kicad_sch (KiCad schematic)
At the start: 17 parts, among them J1 East, J2 West, J4 Display, SW1 Setup, SW2 Reset

Commit message: Migrate Ethernet, SoC, Metering Modules to KiCad6
Parts:
- D1, D2: Manf# (none) -> LTST-C150GKT; part-num (none) -> LTST-C150GKT
- R1, R3: manf# (none) -> RCG1206220RJNEA; part-num (none) -> RCG1206220RJNEA
- R2, R4: part-num (none) -> RCG1206220RJNEA
Changed lines of the file:
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@@
+      (effects (font (size 1.27 1.27)) hide)
+    )
+    (property "Manf#" "LTST-C150GKT" (id 6) (at 119.38 74.93 90)
+      (effects (font (size 1.27 1.27)) hide)
+    )
+    (property "part-num" "LTST-C150GKT" (id 7) (at 119.38 74.93 0)
       (effects (font (size 1.27 1.27)) hide)
     )
@@
       (effects (font (size 1.27 1.27)) hide)
     )
-    (property "Datasheet" "https://www.mouser.de/datasheet/2/427/rcge3-1761759.pdf" (id 3) (at 119.38 63.5 0)
+    (property "Datasheet" "RCG1206220RJNEA" (id 3) (at 119.38 63.5 0)
       (effects (font (size 1.27 1.27)) hide)
     )
@@
     )
     (property "Product" "https://www.mouser.de/ProductDetail/Vishay-Draloric/RCG1206220RJNEA" (id 5) (at 119.38 63.5 0)
+      (effects (font (size 1.27 1.27)) hide)
+    )
+    (property "manf#" "RCG1206220RJNEA" (id 6) (at 119.38 63.5 0)
+      (effects (font (size 1.27 1.27)) hide)
+    )
+    (property "part-num" "RCG1206220RJNEA" (id 7) (at 119.38 63.5 0)
       (effects (font (size 1.27 1.27)) hide)
     )
@@
       (effects (font (size 1.27 1.27)) hide)
     )
+    (property "Manf#" "LTST-C150GKT" (id 6) (at 135.89 74.93 90)
+      (effects (font (size 1.27 1.27)) hide)
+    )
+    (property "part-num" "LTST-C150GKT" (id 7) (at 135.89 74.93 0)
+      (effects (font (size 1.27 1.27)) hide)
+    )
     (pin "1")
     (pin "2")
@@
       (effects (font (size 1.27 1.27)) hide)
     )
-    (property "Datasheet" "https://www.mouser.de/datasheet/2/427/rcge3-1761759.pdf" (id 3) (at 135.89 63.5 0)
+    (property "Datasheet" "RCG1206220RJNEA" (id 3) (at 135.89 63.5 0)
       (effects (font (size 1.27 1.27)) hide)
     )
@@
     )
     (property "Price" "0.08" (id 5) (at 135.89 63.5 0)
+      (effects (font (size 1.27 1.27)) hide)
+    )
+    (property "manf#" "RCG1206220RJNEA" (id 6) (at 135.89 63.5 0)
+      (effects (font (size 1.27 1.27)) hide)
+    )
+    (property "part-num" "RCG1206220RJNEA" (id 7) (at 135.89 63.5 0)
       (effects (font (size 1.27 1.27)) hide)
     )
@@
       (effects (font (size 1.27 1.27)) hide)
     )
+    (property "part-num" "RCG1206220RJNEA" (id 6) (at 71.12 69.85 0)
+      (effects (font (size 1.27 1.27)) hide)
+    )
     (pin "1")
     (pin "2")
@@
       (effects (font (size 1.27 1.27)) hide)
     )
+    (property "part-num" "RCG1206220RJNEA" (id 6) (at 93.98 69.85 0)
+      (effects (font (size 1.27 1.27)) hide)
+    )
