File: smart-meter-module/smart-meter-module.kicad_pcb (KiCad board)
At the start: 2 copper layers, 86 x 31 mm, 25 parts, among them J1 North, J2 RJ12, J3 West, J4 East, J5 RJ12, U3 BA033CC0FP-E2, U4 MAX3486, U5 MAX3486

Commit message: Feature/kicad 6 migration (#2)
* Adjust CI/CD jobs to use KiCad 6

* Migrate panel module project

* Unify KiBot config

* Migrate Ethernet, SoC, Metering Modules to KiCad6

* Change build order to find out more about strange behavior

* Trigger build also on workflow changes

* Try to increase log level to track error

* Switch to KiCad 6 schematic files

* Fix / Ignore Errors in panel module

* Disable cost calculation for now

* Fixing more ERC errors

* Remove outdated files and settings

* Trim further warnings and errors

* Update documentation

* Migrate in-progress projects
Other:
- net class Default removed
