File: electrics/debug-module/debug-module.kicad_sch (KiCad schematic)
At the start: 25 parts, among them J1 East, J2 West, J3 USB_B_Micro, U1 FT231XS, U2 LD1117S33

Commit message: Fix all ERC and DRC warnings during build
Parts:
- removed G1: LOGO, images:grayc-logo-negative, symbol grayc-logo-negative:LOGO
- removed H1: Reset, MountingHole:MountingHole_6.4mm_M6, symbol Mechanical:MountingHole
- removed H2: Status, MountingHole:MountingHole_6.4mm_M6, symbol Mechanical:MountingHole
- added C6, C7: 1nF, Capacitor_SMD:C_1206_3216Metric_Pad1.33x1.80mm_HandSolder, symbol Device:C
- added D5: Power, LED_SMD:LED_1206_3216Metric_Pad1.42x1.75mm_HandSolder, symbol Device:LED
- added D6: Status, LED_SMD:LED_1206_3216Metric_Pad1.42x1.75mm_HandSolder, symbol Device:LED
- added G2: LOGO, symbol grayc-logo-negative:LOGO
- added Q1, Q2: S8050, Package_TO_SOT_SMD:SOT-23, symbol Transistor_BJT:S8050
- added R6, R7: 220R, Resistor_SMD:R_1206_3216Metric_Pad1.30x1.75mm_HandSolder, symbol Device:R
- added SW1: Setup, Button_Switch_SMD:SW_SPST_PTS645, symbol Switch:SW_Push
- added SW2: Reset, Button_Switch_SMD:SW_SPST_PTS645, symbol Switch:SW_Push
- D3: renamed from D?; value LED -> TX
- D4: renamed from D?; value LED -> RX
- J1: renamed from J3; footprint Connector_USB:USB_Micro-B_Wuerth_629105150521 -> Connector_USB:USB_Micro-B_Wuerth_614105150721_Vertical
- R4, R5: renamed from R?; value 10k -> 220R
- gave numbers to parts that had none: 5
- renumbered C1 to C4, C2 to C5, D3 to D7, D4 to D8, G2 to G1, J1 to J2, J2 to J3
Connections:
- net GNDPWR is gone; now on net GND: J1.6 (Shield), J2.14 (Pin_14)
- net +3V3: now also R6.1
- net GND: now also C6.2, C7.2, D5.1 (K), D6.1 (K), SW1.1, SW2.1
- net Panel_Reset: now also C7.1, Q1.3 (C), SW2.2
- net Panel_Setup: now also C6.1, Q2.3 (C), SW1.2
- net Panel_Status: now also R7.1
- net FT_~{DTR}: now reaches U1.1 (~{DTR})
- net FT_~{DTR}: now also Q1.2 (B), Q2.1 (E)
- net FT_~{RTS}: now reaches U1.2 (~{RTS})
- net FT_~{RTS}: now also Q1.1 (E), Q2.2 (B)
- net I2C_SCL: no longer names the net of J2.3 (Pin_3)
- net I2C_SDA: no longer names the net of J2.6 (Pin_6)
- new net: D5.2 (A), R6.2
- new net: D6.2 (A), R7.2
Other:
- note removed: "Bus Mapping"
- moved on the sheet: D3, D4, D7, D8, J2, J3, R4, R5
