File: electrics/debug-module/debug-module.kicad_sch (KiCad schematic)
At the start: 25 parts, among them J1 East, J2 West, J3 USB_B_Micro, U1 FT231XS, U2 LD1117S33

Commit message: INOA-372 Fix autoprogrammer for debug module
Parts:
- removed C? (x2): 47pF, Capacitor_SMD:C_1206_3216Metric_Pad1.33x1.80mm_HandSolder, symbol Device:C
- removed C?: 100nF, Capacitor_SMD:C_1206_3216Metric_Pad1.33x1.80mm_HandSolder, symbol Device:C
- removed D1: BZT52C6V2, Diode_SMD:D_SOD-323_HandSoldering, symbol Device:D_TVS
- removed D2: 1N5819, Diode_SMD:D_SOD-323_HandSoldering, symbol Device:D_Schottky
- removed D3, D4: D_Schottky, Diode_SMD:D_SOD-323_HandSoldering, symbol Device:D_Schottky
- removed D? (x2): LED, LED_SMD:LED_1206_3216Metric_Pad1.42x1.75mm_HandSolder, symbol Device:LED
- removed G2: Logo_Open_Hardware_Small, Symbol:OSHW-Logo2_7.3x6mm_SilkScreen, symbol Graphic:Logo_Open_Hardware_Small
- removed H1: Reset, MountingHole:MountingHole_6.4mm_M6, symbol Mechanical:MountingHole
- removed H2: Status, MountingHole:MountingHole_6.4mm_M6, symbol Mechanical:MountingHole
- removed R? (x2): 10k, Resistor_SMD:R_1206_3216Metric_Pad1.30x1.75mm_HandSolder, symbol Device:R
- removed R? (x2): 27R, Resistor_SMD:R_1206_3216Metric_Pad1.30x1.75mm_HandSolder, symbol Device:R
- added C3: 4u7, Capacitor_SMD:C_1206_3216Metric_Pad1.33x1.80mm_HandSolder, symbol Device:C
- added C4, C5, C6, C7: 100nF, Capacitor_SMD:C_1206_3216Metric_Pad1.33x1.80mm_HandSolder, symbol Device:C
- added C9: 10uF, Capacitor_SMD:C_1206_3216Metric_Pad1.33x1.80mm_HandSolder, symbol Device:C
- added D1: MM3Z6V2T1G, Diode_SMD:D_SOD-123F, symbol Diode:BZT52Bxx
- added D2, D3: 1N5819, Diode_SMD:D_SOD-323_HandSoldering, symbol Diode:1N5819
- added D5: Power, LED_SMD:LED_1206_3216Metric_Pad1.42x1.75mm_HandSolder, symbol Device:LED
- added D6: Status, LED_SMD:LED_1206_3216Metric_Pad1.42x1.75mm_HandSolder, symbol Device:LED
- added D7: TXD, LED_SMD:LED_1206_3216Metric_Pad1.42x1.75mm_HandSolder, symbol Device:LED
- added D8: RXD, LED_SMD:LED_1206_3216Metric_Pad1.42x1.75mm_HandSolder, symbol Device:LED
- added F1: 5V/1A, Fuse:Fuse_1206_3216Metric_Pad1.42x1.75mm_HandSolder, symbol Device:Fuse
- added LOGO1: Logo_Open_Hardware_Small, Symbol:OSHW-Logo_5.7x6mm_SilkScreen, symbol Graphic:Logo_Open_Hardware_Small
- added Q1, Q2: S8050, Package_TO_SOT_SMD:SOT-23-3, symbol Device:Q_NPN_BEC
- added R2: 27R, Resistor_SMD:R_1206_3216Metric_Pad1.30x1.75mm_HandSolder, symbol Device:R
- added R3, R4, R5: 10k, Resistor_SMD:R_1206_3216Metric_Pad1.30x1.75mm_HandSolder, symbol Device:R
- added R6, R7, R8, R9: 220R, Resistor_SMD:R_1206_3216Metric_Pad1.30x1.75mm_HandSolder, symbol Device:R
- added SW1: Reset, Button_Switch_SMD:SW_SPST_PTS645, symbol Switch:SW_SPST
- added SW2: Prog, Button_Switch_SMD:SW_SPST_PTS645, symbol Switch:SW_SPST
- C1: value 100nF -> 47pF; #manf (none) -> C1206C470F3HACTU; #mouser (none) -> 80-C1206C470F3HACTU
- C2: value 10uF -> 47pF; #manf (none) -> C1206C470F3HACTU; #mouser (none) -> 80-C1206C470F3HACTU
- G1: Price 0 -> (none); Product N/A -> (none); now left out of the parts list
- J1, J2: #manf (none) -> 801-83-014-10-001101; #mouser (none) -> 437-8018301410001101
- J3: value USB_B_Micro -> USB; footprint Connector_USB:USB_Micro-B_Wuerth_629105150521 -> Connector_USB:USB_Micro-B_Wuerth_614105150721_Vertical_CircularHoles; #manf (none) -> 614105150721; #mouser (none) -> 710-614105150721
- R1: value 10k -> 27R; #manf (none) -> CRCW120627R0JNEA; #mouser (none) -> 71-CRCW1206J-27-E3
- U1: #manf (none) -> FT231XS-U; #mouser (none) -> 895-FT231XS-U
- U2: #manf (none) -> LD1117S33CTR; #mouser (none) -> 511-LD1117S33C
Connections:
- net GNDPWR is gone; now on net GND: J1.14 (Pin_14), J3.6 (Shield)
- net +3V3: now also C3.1, C4.1, C5.1, C9.1, D3.2 (A), R6.2, R8.2, R9.2; no longer C2.1
- net GND: now also J1.1 (Pin_1), C3.2, C4.2, C5.2, C6.2, C7.2, C9.2, D1.2 (A), D5.1 (K), D6.1 (K), R3.1, SW1.1 (A), SW2.1 (A); no longer R1.2
- net RX_LED: now also D8.1 (K)
- net TX_LED: now also D7.1 (K)
- net at J2.1 (Pin_1): now also D3.1 (K)
- net FT_~{DTR}: now reaches U1.1 (~{DTR})
- net FT_~{DTR}: now also Q1.2 (E), R5.2
- net at U1.11 (USBDP): now also R2.1
- net at U1.12 (USBDM): now also R1.1
- net at U1.13 (3V3OUT), U1.14 (~{RESET}), U1.3 (VCCIO): now also C6.1
- net FT_~{RTS}: now reaches U1.2 (~{RTS})
- net FT_~{RTS}: now also Q2.2 (E), R4.2
- net at U2.3 (VI): now also C7.1, D2.1 (K); no longer C1.1
- net at J3.1 (VBUS): now also F1.1; no longer R1.1
- net I2C_SCL: no longer names the net of J1.3 (Pin_3)
- net I2C_SDA: no longer names the net of J1.6 (Pin_6)
- net Panel_Reset renamed Chip_PU
- net Chip_PU: now also Q2.3 (C), SW1.2 (B)
- net Panel_Setup renamed IO0
- net IO0: now also Q1.3 (C), SW2.2 (B)
- net Panel_Status renamed IO13
- net IO13: now also R7.2
- net USB_DM renamed D-
- net D-: now also C1.1, R1.2
- net USB_DP renamed D+
- net D+: now also C2.1, R2.2
- new net: D7.2 (A), R8.1
- new net: Q1.1 (B), R4.1
- new net: Q2.1 (B), R5.1
- new net: D5.2 (A), R6.1
- new net: D6.2 (A), R7.1
- new net: D8.2 (A), R9.1
- new net: D1.1 (K), D2.2 (A), F1.2, R3.2
Other:
- note removed: "Bus Mapping"
- title: Satellite Panel -> Satellite Debug Panel
- moved on the sheet: J1, J2
