File: electrics/ethernet-extension/ethernet-extension.kicad_pcb (KiCad board)
At the start: 2 copper layers, 56 x 30.4 mm, 44 parts, among them J1 Wuerth_7499010121A, J2 East, J3 West, U1 W5500, Y1 25MHz

Commit message: Fix all ERC and DRC warnings during build
Connections:
- net TD+ renamed TXP
- net TD- renamed TXN
