File: electrics/soc-module/soc-module.kicad_sch (KiCad schematic)
At the start: 19 parts, among them J1 Micro_SD, J2 West, J3 East, U1 ATECC608A-SSHDA, U2 DS3231MZ, U3 ESP32-WROVER-IE-16MB

Commit message: INOA-372 Fix out of stock components in SoC module
Parts:
- R1, R2, R3, R4, R5: manf# CR0603AFX-1002EAS -> CR1206JW-103ELF; mouser# 652-CR0603AFX1002EAS -> 652-CR1206JW-103ELF
Changed lines of the file:
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@@
       (effects (font (size 1.27 1.27)) hide)
     )
-    (property "manf#" "CR0603AFX-1002EAS" (id 6) (at 36.83 38.1 0)
-      (effects (font (size 1.27 1.27)) hide)
-    )
-    (property "mouser#" "652-CR0603AFX1002EAS" (id 7) (at 36.83 38.1 0)
+    (property "manf#" "CR1206JW-103ELF" (id 6) (at 36.83 38.1 0)
+      (effects (font (size 1.27 1.27)) hide)
+    )
+    (property "mouser#" "652-CR1206JW-103ELF" (id 7) (at 36.83 38.1 0)
       (effects (font (size 1.27 1.27)) hide)
     )
@@
       (effects (font (size 1.27 1.27)) hide)
     )
-    (property "manf#" "CR0603AFX-1002EAS" (id 6) (at 36.83 30.48 0)
-      (effects (font (size 1.27 1.27)) hide)
-    )
-    (property "mouser#" "652-CR0603AFX1002EAS" (id 7) (at 36.83 30.48 0)
+    (property "manf#" "CR1206JW-103ELF" (id 6) (at 36.83 30.48 0)
+      (effects (font (size 1.27 1.27)) hide)
+    )
+    (property "mouser#" "652-CR1206JW-103ELF" (id 7) (at 36.83 30.48 0)
       (effects (font (size 1.27 1.27)) hide)
     )
@@
       (effects (font (size 1.27 1.27)) hide)
     )
-    (property "manf#" "CR0603AFX-1002EAS" (id 6) (at 36.83 45.72 0)
-      (effects (font (size 1.27 1.27)) hide)
-    )
-    (property "mouser#" "652-CR0603AFX1002EAS" (id 7) (at 36.83 45.72 0)
+    (property "manf#" "CR1206JW-103ELF" (id 6) (at 36.83 45.72 0)
+      (effects (font (size 1.27 1.27)) hide)
+    )
+    (property "mouser#" "652-CR1206JW-103ELF" (id 7) (at 36.83 45.72 0)
       (effects (font (size 1.27 1.27)) hide)
     )
@@
       (effects (font (size 1.27 1.27)) hide)
     )
-    (property "manf#" "CR0603AFX-1002EAS" (id 6) (at 36.83 53.34 0)
-      (effects (font (size 1.27 1.27)) hide)
-    )
-    (property "mouser#" "652-CR0603AFX1002EAS" (id 7) (at 36.83 53.34 0)
+    (property "manf#" "CR1206JW-103ELF" (id 6) (at 36.83 53.34 0)
+      (effects (font (size 1.27 1.27)) hide)
+    )
+    (property "mouser#" "652-CR1206JW-103ELF" (id 7) (at 36.83 53.34 0)
       (effects (font (size 1.27 1.27)) hide)
     )
@@
       (effects (font (size 1.27 1.27)) hide)
     )
-    (property "manf#" "CR0603AFX-1002EAS" (id 6) (at 36.83 60.96 0)
-      (effects (font (size 1.27 1.27)) hide)
-    )
-    (property "mouser#" "652-CR0603AFX1002EAS" (id 7) (at 36.83 60.96 0)
-      (effects (font (size 1.27 1.27)) hide)
-    )
+    (property "manf#" "CR1206JW-103ELF" (id 6) (at 36.83 60.96 0)
+      (effects (font (size 1.27 1.27)) hide)
+    )
+    (property "mouser#" "652-CR1206JW-103ELF" (id 7) (at 36.83 60.96 0)
+      (effects (font (size 1.27 1.27)) hide)
+    )
