File: electrics/development-board/USB_Interface.kicad_sch (KiCad schematic)
At the start: 24 parts, among them J3 USB_B, U2 FT2232HL, U3 93C46-WMN6TP, Y1 12MHz

Commit message: INOA-372 Rename Fab and Dev board
Connections:
- net +3V3: no longer FB1.1, FB2.2, U3.8 (VCC)
- net EECLK: no longer U3.2 (CLK)
- net EECS: no longer U3.1 (CS)
- net EEDATA: no longer U3.3 (DI)
- net GND: no longer U3.5 (GND)
- net at C10.1, C11.1, U2.4 (VPHY): no longer FB2.1
- net at C12.1, C13.1, U2.9 (VPLL): no longer FB1.2
- net at R6.2, R7.1: no longer U3.4 (DO)
- net at R8.2: no longer U3.6 (ORG)
