File: electrics/pc-board/USB_Interface.kicad_sch (KiCad schematic)
At the start: 24 parts, among them J3 USB_B, U2 FT2232HL, U3 93C46-WMN6TP, Y1 12MHz

Commit message: INOA-372 Rename Fab and Dev board
Connections:
- net +3V3: now also FB1.1, FB2.2, U3.8 (VCC)
- net EECLK: now also U3.2 (CLK)
- net EECS: now also U3.1 (CS)
- net EEDATA: now also U3.3 (DI)
- net GND: now also U3.5 (GND)
- net at C10.1, C11.1, U2.4 (VPHY): now also FB2.1
- net at C12.1, C13.1, U2.9 (VPLL): now also FB1.2
- net at R6.2, R7.1: now also U3.4 (DO)
- net at R8.2: now also U3.6 (ORG)
